Commit message: Second version

File: src/rotors_simulator/rotors_description/urdf/haptic_drone_base.xacro (robot description, xacro)
@@ -24,9 +24,9 @@
   </xacro:if>
   <xacro:include filename="$(find rotors_description)/urdf/nano17.urdf.xacro" />
-  <!-- Macro to add the force vector arrow
-  <xacro:macro name="arrow_plugin">
+  <!-- Macro to add the force vector arrow -->
+  <!--<xacro:macro name="arrow_plugin">-->
     <gazebo>
-      <plugin name="gazebo_visual_plugin" filename="librotors_gazebo_visual_plugin.so" />
+      <plugin name="force_vector" filename="libgazebo_force_vector_visual.so" />
     </gazebo>
-  </xacro:macro>-->
+  <!--</xacro:macro>-->
 </robot>

File: src/rotors_simulator/rotors_description/urdf/models.urdf.xacro (robot description, xacro)
@@ -22,9 +22,9 @@
 		<inertial>
 			<mass value="0.00907"/>
-			<origin xyz="0 0 0.00725"  />
+			<!--<origin xyz="0 0 0.00725"  />-->
+			<origin xyz="0 0 0"  />
 			<xacro:cylinder_inertia_def radius="0.0085" length="0.0145" mass="0.00907"/>
 		</inertial>
 		<visual>
-			<!-- origin xyz="0 0 0.00725" rpy="0 0 0"/ -->
 			<origin xyz="0 0 0" rpy="0 0 0"/>
 			<geometry>
@@ -34,5 +34,6 @@
 		</visual>
 		<collision>
-			<origin xyz="0 0 0.00725" rpy="0 0 0"/>
+			<!--<origin xyz="0 0 0.00725" rpy="0 0 0"/>-->
+			<origin xyz="0 0 0" rpy="0 0 0"/>
 			<geometry>
 				<cylinder radius="0.0085" length="0.0145"/>
@@ -42,11 +43,12 @@
 <xacro:property name="nano17_platform">
 		<inertial>
-			<mass value="0.002"/>
-			<origin xyz="0 0 0.0025"  />
+			<mass value="0.000"/>
+			<!--<origin xyz="0 0 0.0025"  />-->
+			<origin xyz="0 0 0"  />
 			<xacro:cylinder_inertia_def radius="0.0085" length="0.005" mass="0.002"/>
 		</inertial>
 		<visual>
-			<!-- origin xyz="0 0 0.00725" rpy="0 0 0"/ -->
-			<origin xyz="0 0 0.0025" rpy="0 0 0"/>
+			<!--<origin xyz="0 0 0.0025" rpy="0 0 0"/>-->
+			<origin xyz="0 0 0" rpy="0 0 0"/>
 			<geometry>
 				<cylinder radius="0.0085" length="0.005"/>
@@ -54,5 +56,6 @@
 		</visual>
 		<collision>
-			<origin xyz="0 0 0.0025" rpy="0 0 0"/>
+			<!--<origin xyz="0 0 0.0025" rpy="0 0 0"/>-->
+			<origin xyz="0 0 0" rpy="0 0 0"/>
 			<geometry>
 				<cylinder radius="0.0085" length="0.005"/>
@@ -61,5 +64,6 @@
 	</xacro:property>
 	<xacro:property name="nano17_measure_frame">
-		<origin xyz="0 0 0.0145" rpy="0 0 0"/>
+		<!--<origin xyz="0 0 0.0145" rpy="0 0 0"/>-->
+		<origin xyz="0 0 0" rpy="0 0 0"/>
 	</xacro:property>
 </robot>

File: src/rotors_simulator/rotors_description/urdf/nano17.urdf.xacro (robot description, xacro)
@@ -4,5 +4,5 @@
 	<xacro:include filename="$(find rotors_description)/urdf/ft_sensor.urdf.xacro"/>
 	<xacro:ft_sensor parent="haptic_drone/base_link" name="FT_sensor" type="nano17">
-		<origin xyz="0 0 0" rpy="0 0 0"/>
+		<origin xyz="0 0 -0.02" rpy="0 0 0"/>
 	</xacro:ft_sensor>
 </robot>

File: src/structure_haptic_drone/urdf/structure_haptic_drone.urdf (robot description, URDF)
Before this commit: robot structure_haptic_drone, 5 links, 5 joints
Joints:
- joint cage_joint: parent haptic_drone/base_link -> FT_sensor_nano17_measure

File: src/structure_haptic_drone/urdf/vertical_obstacle_higher.xacro (robot description, xacro)
@@ -6,5 +6,5 @@
   <!-- Obstacle description -->
   <m_link_box name="${link_00_name}"
-              origin_rpy="0 0 0" origin_xyz="0.85 -0.7 2.0"
+              origin_rpy="0 0 0" origin_xyz="0.85 -0.8 2.0"
               mass="1000"
               ixx="800.0" ixy="0" ixz="0"
@@ -14,5 +14,5 @@
   <m_joint name="${link_00_name}_${link_01_name}_joint" type="revolute"
            axis_xyz="1 0 0"
-           origin_rpy="0 0 0" origin_xyz="0.85 -0.45 2.75"
+           origin_rpy="0 0 0" origin_xyz="0.85 -0.55 2.75"
            parent="${link_00_name}" child="${link_01_name}"
            limit_e="1000" limit_l="-1.3" limit_u="1.3" limit_v="0.5"
