Commit message: Low stiffness obstacles

File: src/structure_haptic_drone/urdf/obstacle_link_joint.xacro (robot description, xacro)
@@ -6,4 +6,14 @@
       <limit effort="${limit_e}" lower="${limit_l}" upper="${limit_u}" velocity="${limit_v}" />
       <dynamics damping="${damping}" friction="${friction}" />
+      <origin rpy="${origin_rpy}" xyz="${origin_xyz}" />
+      <parent link="${parent}" />
+      <child link="${child}" />
+    </joint>
+  </xacro:macro>
+  <xacro:macro name="k_joint" params="name type axis_xyz origin_rpy origin_xyz parent child limit_e limit_l limit_u limit_v damping friction spring_k spring_ref">
+    <joint name="${name}" type="${type}">
+      <axis xyz="${axis_xyz}" />
+      <limit effort="${limit_e}" lower="${limit_l}" upper="${limit_u}" velocity="${limit_v}" />
+      <dynamics damping="${damping}" friction="${friction}" spring_reference="${spring_ref}" spring_stiffness="${spring_k}" />
       <origin rpy="${origin_rpy}" xyz="${origin_xyz}" />
       <parent link="${parent}" />

File: src/structure_haptic_drone/urdf/vertical_obstacle.xacro (robot description, xacro)
@@ -12,13 +12,13 @@
               izz="800.0"
               size="1.5 0.5 4.0" />
-  <m_joint name="${link_00_name}_${link_01_name}_joint" type="revolute"
+  <m_joint name="branch_joint" type="revolute"
            axis_xyz="1 0 0"
-           origin_rpy="0 0 0" origin_xyz="0.75 2.1 2.0"
+           origin_rpy="0 0 0" origin_xyz="0.75 2.1 1.75"
            parent="${link_00_name}" child="${link_01_name}"
            limit_e="1000" limit_l="-1.3" limit_u="1.3" limit_v="0.5"
-           damping="0.1" friction="0.1" />
+           damping="0.01" friction="0.01" />
   <m_link_box name="${link_01_name}"
               origin_rpy="0 0 0" origin_xyz="0 -0.75 0"
-              mass="0.3"
+              mass="0.1"
               ixx="0.01" ixy="0" ixz="0"
               iyy="0.01" iyz="0"
@@ -39,7 +39,7 @@
   <gazebo>
     <plugin name="joint_spring" filename="libgazebo_joint_torsional_spring.so">
-      <kx>50</kx>
-      <set_point>0.0</set_point>
-      <joint>${link_00_name}_${link_01_name}_joint</joint>
+      <kx>2</kx>
+      <set_point>-0.35</set_point>
+      <joint>branch_joint</joint>
     </plugin>
   </gazebo>

File: src/structure_haptic_drone/urdf/vertical_obstacle_closer.xacro (robot description, xacro)
@@ -14,5 +14,5 @@
   <m_joint name="${link_00_name}_${link_01_name}_joint" type="revolute"
            axis_xyz="1 0 0"
-           origin_rpy="0 0 0" origin_xyz="0.85 -0.35 1.95"
+           origin_rpy="0 0 0" origin_xyz="0.85 -0.35 1.75"
            parent="${link_00_name}" child="${link_01_name}"
            limit_e="1000" limit_l="-0.01" limit_u="1.3" limit_v="0.5"
@@ -20,5 +20,5 @@
   <m_link_box name="${link_01_name}"
               origin_rpy="0 0 0" origin_xyz="0 0.75 0"
-              mass="0.01"
+              mass="0.3"
               ixx="0.01" ixy="0" ixz="0"
               iyy="0.01" iyz="0"
@@ -39,6 +39,6 @@
   <gazebo>
     <plugin name="joint_spring" filename="libgazebo_joint_torsional_spring.so">
-      <kx>0.01</kx>
-      <set_point>0.05</set_point>
+      <kx>100</kx>
+      <set_point>0.01</set_point>
       <joint>${link_00_name}_${link_01_name}_joint</joint>
     </plugin>

File: src/structure_haptic_drone/urdf/vertical_obstacle_higher.xacro (robot description, xacro)
@@ -17,8 +17,8 @@
            parent="${link_00_name}" child="${link_01_name}"
            limit_e="1000" limit_l="-1.3" limit_u="1.3" limit_v="0.5"
-           damping="0.1" friction="0.1" />
+           damping="0.01" friction="0.01" />
   <m_link_box name="${link_01_name}"
               origin_rpy="0 0 0" origin_xyz="0 0.75 0"
-              mass="0.3"
+              mass="0.15"
               ixx="0.01" ixy="0" ixz="0"
               iyy="0.01" iyz="0"
@@ -39,6 +39,6 @@
   <gazebo>
     <plugin name="joint_spring" filename="libgazebo_joint_torsional_spring.so">
-      <kx>100</kx>
-      <set_point>0.05</set_point>
+      <kx>5</kx>
+      <set_point>0.3</set_point>
       <joint>${link_00_name}_${link_01_name}_joint</joint>
     </plugin>
