Commit message: Double control strategy

File: src/structure_haptic_drone/urdf/vertical_obstacle.xacro (robot description, xacro)
@@ -39,9 +39,17 @@
   <gazebo>
     <plugin name="joint_spring" filename="libgazebo_joint_torsional_spring.so">
+      <kx>50</kx>
+      <set_point>-0.0</set_point>
+      <joint>branch_joint</joint>
+    </plugin>
+  </gazebo>
+  <!-- Macro for Torsional Joint Spring Plugin
+  <gazebo>
+    <plugin name="joint_spring" filename="libgazebo_joint_torsional_spring.so">
       <kx>2</kx>
       <set_point>-0.35</set_point>
       <joint>branch_joint</joint>
     </plugin>
-  </gazebo>
+  </gazebo> -->
   <!-- Macro to add the force vector arrow
   <xacro:macro name="arrow_plugin">
@@ -51,76 +59,2 @@
   </xacro:macro>-->
 </robot>
-<!--
-<?xml version="1.0"?>
- <robot xmlns:xacro="http://www.ros.org/wiki/xacro" name="vertical_obstacle">
-    <link name="wall_base">
-    </link>
-    <gazebo reference="wall_base">
-      <gravity>1</gravity>
-    </gazebo>
-  <xacro:macro name="joint_base">
-    <joint name="wall_base_joint" type="fixed">
-        <parent link="wall_base"/>
-        <child link="wall"/>
-        <axis xyz="0 0 1" />
-        <origin xyz="0 0 0" rpy="0 0 0"/>
-    </joint>
-  </xacro:macro>
-  <xacro:macro name="wall">
-   <link name="wall">
-     <inertial>
-       <origin xyz="0 1.0 1.0" />
-       <mass value="100.0" />
-       <inertia  ixx="10.0" ixy="0.0"  ixz="0.0"  iyy="10.0"  iyz="0.0"  izz="10.0" />
-     </inertial>
-     <visual>
-       <origin xyz="0 1.0 1.0"/>
-       <geometry>
-         <box size="1.5 0.5 2.0" />
-        </geometry>
-     </visual>
-     <collision>
-       <origin xyz="0 1.0 1.0"/>
-       <geometry>
-         <box size="1.5 0.5 2.0" />
-       </geometry>
-     </collision>
-   </link>
-   <gazebo reference="wall">
-     <material>Gazebo/Grey</material>
-   </gazebo>
-  </xacro:macro>
-  <xacro:macro name="joint1">
-   <joint name="spring_joint" type="revolute">
-        <parent link="wall_base"/>
-        <child link="branch"/>
-        <axis xyz="0 -1 0" />
-        <origin xyz="0 0 0" rpy="0 0 0"/>
-    </joint>
-  </xacro:macro>
-  <xacro:macro name="branch">
-   <link name="branch">
-     <inertial>
-       <origin xyz="3.0 1.0 1.0" />
-       <mass value="0.1" />
-       <inertia  ixx="0.1" ixy="0.0"  ixz="0.0"  iyy="0.1"  iyz="0.0"  izz="0.1" />
-     </inertial>
-     <visual>
-       <origin xyz="0 1.0 1.0"/>
-       <geometry>
-         <box size="1.5 1.5 0.05" />
-        </geometry>
-     </visual>
-     <collision>
-       <origin xyz="0 1.0 1.0"/>
-       <geometry>
-         <box size="1.5 1.5 0.05" />
-       </geometry>
-     </collision>
-   </link>
-   <gazebo reference="branch">
-     <material>Gazebo/Grey</material>
-   </gazebo>
-  </xacro:macro>
-</robot>
--->
